Commit message: Fix description

File: clearpath_dual_franka_description/urdf/clearpath_dual_franka.urdf.xacro (robot description, xacro)
@@ -13,12 +13,12 @@
     **arm_0_gripper_origin
     arm_1_parent:=base_link
-    arm_1_ip:=192.168.131.40
+    arm_1_ip:=192.168.131.41
     arm_1_id:=fr3
-    arm_1_name:=arm_0
+    arm_1_name:=arm_1
     arm_1_control:=false
     **arm_1_origin
     arm_1_gripper_enable:=true
-    arm_1_gripper_name:=arm_0_gripper
-    arm_1_gripper_parent:=arm_0_fr3_link8
+    arm_1_gripper_name:=arm_1_gripper
+    arm_1_gripper_parent:=arm_1_fr3_link8
     **arm_1_gripper_origin
     ">
@@ -26,28 +26,16 @@
     <xacro:include filename="$(find clearpath_manipulators_description)/urdf/gripper/franka_gripper.urdf.xacro"/>
     <!-- arm_0 -->
-    <!-- <xacro:franka name="arm_0" parent_link="arm_mount_left_link" robot_ip="192.168.131.40" arm_id="fr3" ros2_control="$(arg arm_0_control)">
-      <origin xyz="0.0 0.0 0.0" rpy="0.0 0.0 0.7854"/>
-    </xacro:franka> -->
     <xacro:franka name="${arm_0_name}" parent_link="${arm_0_parent}" robot_ip="${arm_0_ip}" arm_id="${arm_0_id}" ros2_control="${arm_0_control}">
       <xacro:insert_block name="arm_0_origin"/>
     </xacro:franka>
     <!-- arm_1 -->
-    <!-- <xacro:franka name="arm_1" parent_link="arm_mount_right_link" robot_ip="192.168.131.41" arm_id="fr3" ros2_control="$(arg arm_1_control)">
-      <origin xyz="0.0 0.0 0.0" rpy="0.0 0.0 -0.7854"/>
-    </xacro:franka> -->
     <xacro:franka name="${arm_1_name}" parent_link="${arm_1_parent}" robot_ip="${arm_1_ip}" arm_id="${arm_1_id}" ros2_control="${arm_1_control}">
       <xacro:insert_block name="arm_1_origin"/>
     </xacro:franka>
     <!-- arm_0_gripper -->
-    <!-- <xacro:franka_gripper name="arm_0_gripper" parent_link="arm_0_fr3_link8" arm_id="fr3">
-      <origin xyz="0.0 0.0 0.0" rpy="0.0 0.0 0.0"/>
-    </xacro:franka_gripper> -->
     <xacro:franka_gripper name="${arm_0_gripper_name}" parent_link="${arm_0_gripper_parent}" arm_id="${arm_0_id}">
       <xacro:insert_block name="arm_0_gripper_origin"/>
     </xacro:franka_gripper>
     <!-- arm_1_gripper -->
-    <!-- <xacro:franka_gripper name="arm_1_gripper" parent_link="arm_1_fr3_link8" arm_id="fr3">
-      <origin xyz="0.0 0.0 0.0" rpy="0.0 0.0 0.0"/>
-    </xacro:franka_gripper> -->
     <xacro:franka_gripper name="${arm_1_gripper_name}" parent_link="${arm_1_gripper_parent}" arm_id="${arm_1_id}">
       <xacro:insert_block name="arm_1_gripper_origin"/>
